File: d-ampsch.brd (EAGLE design)
At the start: 125.4 x 138.4 mm, 38 parts

Commit message: wire done
needs more fixes tho
Parts:
- moved C6 122.9 mm to (73.4, 68.1)
- moved C9 121.4 mm to (60.2, 77.2), turned to 90 degrees
- moved C7 117.9 mm to (63.2, 87.4)
- moved C5 110.3 mm to (68.3, 87.4)
- moved R8 103.9 mm to (79.0, 72.4)
- moved R9 101.7 mm to (74.7, 84.8), turned to 90 degrees
- moved R11 79.1 mm to (3.81, 59.7), turned to 180 degrees
- moved R10 75.7 mm to (2.79, 53.6)
- moved R7 62.5 mm to (21.6, 57.1)
- moved R6 59.2 mm to (21.6, 50.8)
- moved D5 52.0 mm to (12.1, 42.5), turned to 90 degrees
- moved U$14 43.3 mm to (69.6, 77.1)
- moved D4 32.5 mm to (5.08, 42.5), turned to 90 degrees
- moved D3 30.7 mm to (92.2, 70.4), turned to 0 degrees
- moved C10 25.4 mm to (24.6, 68.3)
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Routing:
- net GND: track 12.7 -> 128.5 mm, vias 0 -> 29
- net +3V3: track 0.00 -> 84.3 mm, vias 0 -> 4
- net I2S1_SD: track 0.00 -> 75.0 mm
- net I2S1_CK: track 0.00 -> 74.2 mm
- net I2S1_WS: track 0.00 -> 73.0 mm
- net PWM: track 15.1 -> 67.7 mm, vias 0 -> 2
- net PWMINV: track 12.5 -> 56.3 mm
- net N$4: track 0.00 -> 35.4 mm
- net N$15: track 0.00 -> 30.3 mm, vias 0 -> 2
- net CON-VDD: track 0.00 -> 29.2 mm
- net N$10: track 0.00 -> 28.3 mm
- net N$13: track 0.00 -> 27.7 mm, vias 0 -> 2
- net NRST: track 0.00 -> 26.4 mm, vias 0 -> 2
- net N$14: track 0.00 -> 25.0 mm
- net N$16: track 0.00 -> 23.5 mm
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- added copper zone on layer 16, net GND
Other:
- board size 125.4 x 138.4 mm -> 99.5 x 97.4 mm
- board text added: "HBRIDGE-DAMP V2.0 Benjamin"

Commit message: mostly finished
might have to fix stuff
Parts:
- moved R10 5.33 mm to (2.79, 48.3)
- moved R11 2.54 mm to (3.81, 62.2), turned to 270 degrees
Connections:
- removed net CON-VDD: C5.1, C6.1, C7.1, U$14.24, U$14.48
- removed net CON-VDDA: C8.1, C9.1, U$14.9
- net +3V3: now also C5.1, C6.1, C7.1, C8.1, C9.1, U$14.24, U$14.48, U$14.9
Routing:
- net +3V3: track 84.3 -> 131.2 mm
- net CON-VDD: track 29.2 -> 0.00 mm
- net LOAD-RIGHT: track 85.3 -> 69.9 mm
- net GND: track 128.5 -> 139.0 mm, vias 29 -> 30
- net CON-VDDA: track 10.3 -> 0.00 mm
- net LOAD-LEFT: track 50.8 -> 57.0 mm
- net N$16: track 23.5 -> 28.8 mm
- net N$2: track 8.84 -> 5.61 mm
- net N$8: track 28.5 -> 29.6 mm
