File: d-ampsch.brd (EAGLE design)
At the start: 99.5 x 97.4 mm, 38 parts

Commit message: fixed stuff
Routing:
- net LOAD-LEFT: track 57.0 -> 52.5 mm
- net I2S1_SD: track 75.0 -> 76.0 mm
- net I2S1_WS: track 73.0 -> 73.7 mm
- net I2S1_CK: track 74.2 -> 74.7 mm
