File: d-ampsch.sch (EAGLE design)
At the start: 38 parts

Commit message: mostly finished
might have to fix stuff
Connections:
- removed net CON-VDD: C5.P$1, C6.P$1, C7.P$1, U$14.VDD@24, U$14.VDD@48
- removed net CON-VDDA: C8.P$1, C9.P$1, U$14.VDDA
- net +3V3: now also C5.P$1, C6.P$1, C7.P$1, C8.P$1, C9.P$1, U$14.VDD@24, U$14.VDD@48, U$14.VDDA
Changed lines of the file:
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@@
 <layers>
 <layer number="1" name="Top" color="4" fill="1" visible="no" active="no"/>
+<layer number="2" name="Route2" color="1" fill="3" visible="no" active="no"/>
+<layer number="3" name="Route3" color="4" fill="3" visible="no" active="no"/>
+<layer number="4" name="Route4" color="1" fill="4" visible="no" active="no"/>
+<layer number="5" name="Route5" color="4" fill="4" visible="no" active="no"/>
+<layer number="6" name="Route6" color="1" fill="8" visible="no" active="no"/>
+<layer number="7" name="Route7" color="4" fill="8" visible="no" active="no"/>
+<layer number="8" name="Route8" color="1" fill="2" visible="no" active="no"/>
+<layer number="9" name="Route9" color="4" fill="2" visible="no" active="no"/>
+<layer number="10" name="Route10" color="1" fill="7" visible="no" active="no"/>
+<layer number="11" name="Route11" color="4" fill="7" visible="no" active="no"/>
+<layer number="12" name="Route12" color="1" fill="5" visible="no" active="no"/>
+<layer number="13" name="Route13" color="4" fill="5" visible="no" active="no"/>
+<layer number="14" name="Route14" color="1" fill="6" visible="no" active="no"/>
+<layer number="15" name="Route15" color="4" fill="6" visible="no" active="no"/>
 <layer number="16" name="Bottom" color="1" fill="1" visible="no" active="no"/>
 <layer number="17" name="Pads" color="2" fill="1" visible="no" active="no"/>
@@
 <part name="C9" library="amplib" deviceset="C-10NF" device="" package3d_urn="urn:adsk.eagle:package:17050553/1" value="10NF"/>
 <part name="C8" library="amplib" deviceset="C-1UF-NP" device="C-1UF-NP" package3d_urn="urn:adsk.eagle:package:17050632/1" value="1UF"/>
+<part name="U$1" library="amplib" deviceset="B-BATTERY" device="BATTERYCONN" package3d_urn="urn:adsk.eagle:package:17097127/1"/>
+<part name="VDD1" library="supply1" library_urn="urn:adsk.eagle:library:371" deviceset="VDD" device=""/>
+<part name="+3V7" library="supply1" library_urn="urn:adsk.eagle:library:371" deviceset="+3V3" device=""/>
+<part name="+3V8" library="supply1" library_urn="urn:adsk.eagle:library:371" deviceset="+3V3" device=""/>
+<part name="+3V9" library="supply1" library_urn="urn:adsk.eagle:library:371" deviceset="+3V3" device=""/>
 <part name="+3V5" library="supply1" library_urn="urn:adsk.eagle:library:371" deviceset="+3V3" device=""/>
 <part name="+3V6" library="supply1" library_urn="urn:adsk.eagle:library:371" deviceset="+3V3" device=""/>
-<part name="U$1" library="amplib" deviceset="B-BATTERY" device="BATTERYCONN" package3d_urn="urn:adsk.eagle:package:17097127/1"/>
-<part name="VDD1" library="supply1" library_urn="urn:adsk.eagle:library:371" deviceset="VDD" device=""/>
 </parts>
 <sheets>
@@
 <attribute name="VALUE" x="81.28" y="106.68" size="1.27" layer="96" rot="R270"/>
 </instance>
-<instance part="+3V5" gate="G$1" x="104.14" y="137.16" smashed="yes" rot="R270">
-<attribute name="VALUE" x="99.06" y="139.7" size="1.778" layer="96"/>
-</instance>
-<instance part="+3V6" gate="G$1" x="91.44" y="109.22" smashed="yes" rot="R270">
-<attribute name="VALUE" x="86.36" y="111.76" size="1.778" layer="96"/>
+<instance part="+3V7" gate="G$1" x="-50.8" y="109.22" smashed="yes">
+<attribute name="VALUE" x="-53.34" y="104.14" size="1.778" layer="96" rot="R90"/>
+</instance>
+<instance part="+3V8" gate="G$1" x="-96.52" y="53.34" smashed="yes" rot="R90">
+<attribute name="VALUE" x="-91.44" y="50.8" size="1.778" layer="96" rot="R180"/>
+</instance>
+<instance part="+3V9" gate="G$1" x="-22.86" y="10.16" smashed="yes" rot="R180">
+<attribute name="VALUE" x="-20.32" y="15.24" size="1.778" layer="96" rot="R270"/>
+</instance>
+<instance part="+3V5" gate="G$1" x="93.98" y="109.22" smashed="yes" rot="R270">
+<attribute name="VALUE" x="88.9" y="111.76" size="1.778" layer="96"/>
+</instance>
+<instance part="+3V6" gate="G$1" x="106.68" y="137.16" smashed="yes" rot="R270">
+<attribute name="VALUE" x="101.6" y="139.7" size="1.778" layer="96"/>
 </instance>
 </instances>
@@
 <pinref part="U$13" gate="G$1" pin="VDD_PADS"/>
 <pinref part="+3V3" gate="G$1" pin="+3V3"/>
-<wire x1="116.84" y1="86.36" x2="116.84" y2="91.44" width="0.1524" layer="91"/>
+<wire x1="116.84" y1="86.36" x2="116.84" y2="88.9" width="0.1524" layer="91"/>
+<wire x1="116.84" y1="88.9" x2="116.84" y2="91.44" width="0.1524" layer="91"/>
+<wire x1="116.84" y1="88.9" x2="116.84" y2="93.98" width="0.1524" layer="91"/>
 </segment>
 <segment>
@@
 <wire x1="-66.04" y1="73.66" x2="-73.66" y2="73.66" width="0.1524" layer="91"/>
 <pinref part="+3V4" gate="G$1" pin="+3V3"/>
+</segment>
+<segment>
+<pinref part="U$14" gate="G$1" pin="VDDA"/>
+<wire x1="-66.04" y1="53.34" x2="-93.98" y2="53.34" width="0.1524" layer="91"/>
+<pinref part="+3V8" gate="G$1" pin="+3V3"/>
+</segment>
+<segment>
+<pinref part="U$14" gate="G$1" pin="VDD@48"/>
+<wire x1="-50.8" y1="88.9" x2="-50.8" y2="106.68" width="0.1524" layer="91"/>
+<pinref part="+3V7" gate="G$1" pin="+3V3"/>
+</segment>
+<segment>
+<pinref part="U$14" gate="G$1" pin="VDD@24"/>
+<wire x1="-22.86" y1="30.48" x2="-22.86" y2="12.7" width="0.1524" layer="91"/>
+<pinref part="+3V9" gate="G$1" pin="+3V3"/>
+</segment>
+<segment>
+<pinref part="C5" gate="G$1" pin="P$1"/>
+<wire x1="73.66" y1="134.62" x2="73.66" y2="137.16" width="0.1524" layer="91"/>
+<pinref part="C6" gate="G$1" pin="P$1"/>
+<wire x1="73.66" y1="137.16" x2="83.82" y2="137.16" width="0.1524" layer="91"/>
+<wire x1="83.82" y1="137.16" x2="83.82" y2="134.62" width="0.1524" layer="91"/>
+<pinref part="C7" gate="G$1" pin="P$1"/>
+<wire x1="83.82" y1="137.16" x2="96.52" y2="137.16" width="0.1524" layer="91"/>
+<wire x1="96.52" y1="137.16" x2="96.52" y2="134.62" width="0.1524" layer="91"/>
+<junction x="83.82" y="137.16"/>
+<wire x1="96.52" y1="137.16" x2="104.14" y2="137.16" width="0.1524" layer="91"/>
+<junction x="96.52" y="137.16"/>
+<pinref part="+3V6" gate="G$1" pin="+3V3"/>
+</segment>
+<segment>
+<pinref part="C9" gate="G$1" pin="P$1"/>
+<wire x1="73.66" y1="106.68" x2="73.66" y2="109.22" width="0.1524" layer="91"/>
+<wire x1="73.66" y1="109.22" x2="86.36" y2="109.22" width="0.1524" layer="91"/>
+<pinref part="C8" gate="G$1" pin="P$1"/>
+<wire x1="86.36" y1="109.22" x2="86.36" y2="106.68" width="0.1524" layer="91"/>
+<junction x="86.36" y="109.22"/>
+<pinref part="+3V5" gate="G$1" pin="+3V3"/>
+<wire x1="86.36" y1="109.22" x2="91.44" y2="109.22" width="0.1524" layer="91"/>
 </segment>
 </net>
@@
 </segment>
 </net>
-<net name="CON-VDD" class="0">
-<segment>
-<pinref part="U$14" gate="G$1" pin="VDD@48"/>
-<wire x1="-50.8" y1="88.9" x2="-50.8" y2="104.14" width="0.1524" layer="91"/>
-<label x="-50.8" y="104.14" size="1.778" layer="95" rot="R90" xref="yes"/>
-</segment>
-<segment>
-<pinref part="U$14" gate="G$1" pin="VDD@24"/>
-<wire x1="-22.86" y1="30.48" x2="-22.86" y2="15.24" width="0.1524" layer="91"/>
-<label x="-22.86" y="15.24" size="1.778" layer="95" rot="R270" xref="yes"/>
-</segment>
-<segment>
-<pinref part="C5" gate="G$1" pin="P$1"/>
-<wire x1="73.66" y1="134.62" x2="73.66" y2="137.16" width="0.1524" layer="91"/>
-<pinref part="C6" gate="G$1" pin="P$1"/>
-<wire x1="73.66" y1="137.16" x2="81.28" y2="137.16" width="0.1524" layer="91"/>
-<wire x1="81.28" y1="137.16" x2="83.82" y2="137.16" width="0.1524" layer="91"/>
-<wire x1="83.82" y1="137.16" x2="83.82" y2="134.62" width="0.1524" layer="91"/>
-<pinref part="C7" gate="G$1" pin="P$1"/>
-<wire x1="83.82" y1="137.16" x2="96.52" y2="137.16" width="0.1524" layer="91"/>
-<wire x1="96.52" y1="137.16" x2="96.52" y2="134.62" width="0.1524" layer="91"/>
-<junction x="83.82" y="137.16"/>
-<wire x1="81.28" y1="137.16" x2="81.28" y2="139.7" width="0.1524" layer="91"/>
-<junction x="81.28" y="137.16"/>
-<label x="81.28" y="139.7" size="1.778" layer="95" rot="R90" xref="yes"/>
-<wire x1="96.52" y1="137.16" x2="101.6" y2="137.16" width="0.1524" layer="91"/>
-<junction x="96.52" y="137.16"/>
-<pinref part="+3V5" gate="G$1" pin="+3V3"/>
-</segment>
-</net>
-<net name="CON-VDDA" class="0">
-<segment>
-<pinref part="U$14" gate="G$1" pin="VDDA"/>
-<wire x1="-66.04" y1="53.34" x2="-91.44" y2="53.34" width="0.1524" layer="91"/>
-<label x="-91.44" y="53.34" size="1.778" layer="95" rot="R180" xref="yes"/>
-</segment>
-<segment>
-<pinref part="C9" gate="G$1" pin="P$1"/>
-<wire x1="73.66" y1="106.68" x2="73.66" y2="109.22" width="0.1524" layer="91"/>
-<wire x1="73.66" y1="109.22" x2="86.36" y2="109.22" width="0.1524" layer="91"/>
-<pinref part="C8" gate="G$1" pin="P$1"/>
-<wire x1="86.36" y1="109.22" x2="86.36" y2="106.68" width="0.1524" layer="91"/>
-<wire x1="73.66" y1="109.22" x2="71.12" y2="109.22" width="0.1524" layer="91"/>
-<junction x="73.66" y="109.22"/>
-<label x="71.12" y="109.22" size="1.778" layer="95" rot="R180" xref="yes"/>
-<wire x1="86.36" y1="109.22" x2="88.9" y2="109.22" width="0.1524" layer="91"/>
-<junction x="86.36" y="109.22"/>
-<pinref part="+3V6" gate="G$1" pin="+3V3"/>
-</segment>
-</net>
